File: kicad/esp8266.sch (KiCad schematic (older format))
At the start: 6 parts, among them J2 Conn_Coaxial_Power, Q1 BSP75, U1 ESP-12E, U4 MS5637, U5 PCA9685PW, U6 Si7020-A20

Commit message: improve kicad
Parts:
- added D? (x2): D_Schottky, symbol Device:D_Schottky
- added J3: CONN FT232RL, Connector_PinHeader_2.54mm:PinHeader_1x06_P2.54mm_Vertical, symbol Connector:Conn_01x06_Female
- added J4, J5: RJ12, Connector_RJ:RJ12_Amphenol_54601, symbol Connector:RJ12
- added Q2, Q3, Q4: BSP75, Package_TO_SOT_SMD:SOT-223-3_TabPin2, symbol esp8266-rescue:BSP75-lpatiny
- added R7, R?: 10k, Resistor_SMD:R_0805_2012Metric_Pad1.15x1.40mm_HandSolder, symbol Device:R
- added R?: 4.7k, Resistor_SMD:R_0805_2012Metric_Pad1.15x1.40mm_HandSolder, symbol Device:R
- added SW1, SW?: SW_Push, digikey-footprints:Switch_Tactile_SMD_6x6mm, symbol Switch:SW_Push
- Q1: symbol lpatiny:BSP75 -> esp8266-rescue:BSP75-lpatiny
- U4: symbol ms5637:MS5637 -> esp8266-rescue:MS5637-ms5637
Connections:
- net labels added: +12V, CTS, DTR, Onewire, RX, SCL, SDA, TX, VBAT, VCC-FTDI, VCC_FTDI, V_PROBE, V_STATUS
- wire segments 8 -> 49
Other:
- note added: "CTS"
- note added: "DTR"
- note added: "GND"
- note added: "RX"
- note added: "TX"
- note added: "VCC"
- note added: "ab"

Commit message: updates
Parts:
- removed U5: PCA9685PW, Package_SO:TSSOP-28_4.4x9.7mm_P0.65mm, symbol Driver_LED:PCA9685PW
- added J6, J7: Onewire, Connector_Audio:Jack_3.5mm_Ledino_KB3SPRS_Horizontal, symbol Onewire:Onewire
- added R8: 10k, Resistor_SMD:R_0805_2012Metric_Pad1.15x1.40mm_HandSolder, symbol Device:R
- D3, D4: renamed from D?; footprint (none) -> Diode_SMD:D_SOD-123
- Q1, Q2, Q3, Q4: symbol esp8266-rescue:BSP75-lpatiny -> BSP75:BSP75
- SW1: value SW_Push -> RESET
- SW2: renamed from SW?; value SW_Push -> PROG
- U4: symbol esp8266-rescue:MS5637-ms5637 -> ms5637:MS5637
- gave numbers to parts that had none: 2
Connections:
- net labels added: ADC, EN, IO2, PWM_R, RST
- net labels removed: Onewire, V_PROBE, V_STATUS
- wire segments 49 -> 53
Other:
- note added: "Onewire\n"
- note added: "USED BY FLASH"

Commit message: add 18B20 on board
Parts:
- added U7: DS18B20, Package_TO_SOT_THT:TO-92_Inline, symbol Sensor_Temperature:DS18B20
- U4: footprint (none) -> libs:MS5637
Connections:
- net labels added: IO12, IO13, IO14, IO15
- net labels removed: PWM_R, VCC-FTDI
Changed lines of the file:
@@
 F 0 "U4" H 7700 3287 60  0000 C CNN
 F 1 "MS5637" H 7700 3181 60  0000 C CNN
-F 2 "" H 7400 2900 60  0001 C CNN
+F 2 "libs:MS5637" H 7400 2900 60  0001 C CNN
 F 3 "" H 7400 2900 60  0000 C CNN
 	1    7700 2950
@@
 $EndComp
 Text Label 1600 4350 0    50   ~ 0
-VCC-FTDI
+VCC_FTDI
 Wire Wire Line
 	1500 4050 1950 4050
@@
 Wire Wire Line
 	5250 5150 5600 5150
-Text Label 5300 4850 0    50   ~ 0
-PWM_R
 Text Notes 5650 4450 0    50   ~ 0
 Onewire\n
@@
 Wire Wire Line
 	5750 4250 6000 4250
+Text Label 5300 4950 0    50   ~ 0
+IO13
+Text Label 5300 5050 0    50   ~ 0
+IO14
+Text Label 5300 5150 0    50   ~ 0
+IO15
+Text Label 5300 4850 0    50   ~ 0
+IO12
+$Comp
+L Sensor_Temperature:DS18B20 U7
+U 1 1 5C3F9182
+P 10000 2950
+F 0 "U7" H 9770 2996 50  0000 R CNN
+F 1 "DS18B20" H 9770 2905 50  0000 R CNN
+F 2 "Package_TO_SOT_THT:TO-92_Inline" H 9000 2700 50  0001 C CNN
+F 3 "http://datasheets.maximintegrated.com/en/ds/DS18B20.pdf" H 9850 3200 50  0001 C CNN
+	1    10000 2950
+	1    0    0    -1
+$EndComp
 $EndSCHEMATC

Commit message: correst bsp75 footprint
Parts:
- added J8: Conn_01x01_Male, symbol Connector:Conn_01x01_Male
- Q1, Q2, Q3, Q4: footprint Package_TO_SOT_SMD:SOT-223-3_TabPin2 -> Package_TO_SOT_SMD:SOT-223
Connections:
- wire segments 53 -> 56
Changed lines of the file:
@@
 L BSP75:BSP75 Q1
 U 1 1 5C3A4B25
-P 9300 3400
-F 0 "Q1" H 9506 3446 50  0000 L CNN
-F 1 "BSP75" H 9506 3355 50  0000 L CNN
-F 2 "Package_TO_SOT_SMD:SOT-223-3_TabPin2" H 9500 3325 50  0001 L CIN
-F 3 "https://www.infineon.com/dgdl/Infineon-BSP129-DS-v01_42-en.pdf?fileId=db3a30433c1a8752013c1fc296d2395f" H 9500 3475 50  0001 L CNN
-	1    9300 3400
+P 9050 3400
+F 0 "Q1" H 9256 3446 50  0000 L CNN
+F 1 "BSP75" H 9256 3355 50  0000 L CNN
+F 2 "Package_TO_SOT_SMD:SOT-223" H 9250 3325 50  0001 L CIN
+F 3 "https://www.infineon.com/dgdl/Infineon-BSP129-DS-v01_42-en.pdf?fileId=db3a30433c1a8752013c1fc296d2395f" H 9250 3475 50  0001 L CNN
+	1    9050 3400
 	1    0    0    -1
 $EndComp
@@
 F 0 "Q2" H 9456 4046 50  0000 L CNN
 F 1 "BSP75" H 9456 3955 50  0000 L CNN
-F 2 "Package_TO_SOT_SMD:SOT-223-3_TabPin2" H 9450 3925 50  0001 L CIN
+F 2 "Package_TO_SOT_SMD:SOT-223" H 9450 3925 50  0001 L CIN
 F 3 "https://www.infineon.com/dgdl/Infineon-BSP129-DS-v01_42-en.pdf?fileId=db3a30433c1a8752013c1fc296d2395f" H 9450 4075 50  0001 L CNN
 	1    9250 4000
@@
 F 0 "Q3" H 9506 4746 50  0000 L CNN
 F 1 "BSP75" H 9506 4655 50  0000 L CNN
-F 2 "Package_TO_SOT_SMD:SOT-223-3_TabPin2" H 9500 4625 50  0001 L CIN
+F 2 "Package_TO_SOT_SMD:SOT-223" H 9500 4625 50  0001 L CIN
 F 3 "https://www.infineon.com/dgdl/Infineon-BSP129-DS-v01_42-en.pdf?fileId=db3a30433c1a8752013c1fc296d2395f" H 9500 4775 50  0001 L CNN
 	1    9300 4700
@@
 F 0 "Q4" H 9556 5396 50  0000 L CNN
 F 1 "BSP75" H 9556 5305 50  0000 L CNN
-F 2 "Package_TO_SOT_SMD:SOT-223-3_TabPin2" H 9550 5275 50  0001 L CIN
+F 2 "Package_TO_SOT_SMD:SOT-223" H 9550 5275 50  0001 L CIN
 F 3 "https://www.infineon.com/dgdl/Infineon-BSP129-DS-v01_42-en.pdf?fileId=db3a30433c1a8752013c1fc296d2395f" H 9550 5425 50  0001 L CNN
 	1    9350 5350
@@
 	1    0    0    -1
 $EndComp
+$Comp
+L power:GND #PWR0132
+U 1 1 5C3FE6C9
+P 9150 3650
+F 0 "#PWR0132" H 9150 3400 50  0001 C CNN
+F 1 "GND" H 9155 3477 50  0000 C CNN
+F 2 "" H 9150 3650 50  0001 C CNN
+F 3 "" H 9150 3650 50  0001 C CNN
+	1    9150 3650
+	1    0    0    -1
+$EndComp
+Wire Wire Line
+	9150 3650 9150 3600
+Wire Wire Line
+	8850 3400 8650 3400
+Text Label 8700 3400 0    50   ~ 0
+IO12
+$Comp
+L Connector:Conn_01x01_Male J8
+U 1 1 5C401F99
+P 9350 3100
+F 0 "J8" H 9323 3030 50  0000 R CNN
+F 1 "Conn_01x01_Male" H 9323 3121 50  0000 R CNN
+F 2 "" H 9350 3100 50  0001 C CNN
+F 3 "~" H 9350 3100 50  0001 C CNN
+	1    9350 3100
+	-1   0    0    1
+$EndComp
+Wire Wire Line
+	9150 3100 9150 3200
 $EndSCHEMATC

Commit message: add test points in kicad
Parts:
- added J10: Green, Connector_Wire:SolderWirePad_1x01_SMD_5x10mm, symbol Connector:Conn_01x01_Male
- added J11: Blue, Connector_Wire:SolderWirePad_1x01_SMD_5x10mm, symbol Connector:Conn_01x01_Male
- added J12: White, Connector_Wire:SolderWirePad_1x01_SMD_5x10mm, symbol Connector:Conn_01x01_Male
- added J13: Conn_01x08_Female, Connector_PinHeader_2.54mm:PinHeader_1x08_P2.54mm_Vertical, symbol Connector:Conn_01x08_Female
- added J9: Pad, Connector_Wire:SolderWirePad_1x01_SMD_5x10mm, symbol Connector:Conn_01x01_Male
- added TP2: I2C, TestPoint:TestPoint_2Pads_Pitch2.54mm_Drill0.8mm, symbol Connector:TestPoint_2Pole
- added TP3: OneWire, TestPoint:TestPoint_2Pads_Pitch2.54mm_Drill0.8mm, symbol Connector:TestPoint_2Pole
- added TP?: 3.3V, symbol Connector:TestPoint_2Pole
- added TP?: TestPoint_2Pole, symbol Connector:TestPoint_2Pole
- added TP?: V_OUT, symbol Connector:TestPoint_2Pole
- added TP?: V_BAT, symbol Connector:TestPoint_2Pole
- J8: value Conn_01x01_Male -> Red; footprint (none) -> Connector_Wire:SolderWirePad_1x01_SMD_5x10mm
Connections:
- net labels added: +BATT
- net labels removed: VBAT
- wire segments 56 -> 91

Commit message: add more test points
Parts:
- removed TP2: I2C, TestPoint:TestPoint_2Pads_Pitch2.54mm_Drill0.8mm, symbol Connector:TestPoint_2Pole
- added J14: +12V, Connector_Wire:SolderWirePad_1x01_SMD_5x10mm, symbol Connector:Conn_01x01_Male
- added TP2: Test_i2C, Connector_PinHeader_2.54mm:PinHeader_1x01_P2.54mm_Vertical, symbol Test_points:Test_i2C
- J13: value Conn_01x08_Female -> IO_RGBW
- J2: value Conn_Coaxial_Power -> 5 / 12V
- J4, J5: value RJ12 -> RJ12-I2C; symbol Connector:RJ12 -> rj12:RJ12-I2C
- TP1: renamed from TP?; value TestPoint_2Pole -> 5V; footprint (none) -> TestPoint:TestPoint_2Pads_Pitch2.54mm_Drill0.8mm
- TP4, TP5, TP6: renamed from TP?; footprint (none) -> TestPoint:TestPoint_2Pads_Pitch2.54mm_Drill0.8mm
Connections:
- wire segments 91 -> 111

Commit message: working on routing
Parts:
- TP2: footprint Connector_PinHeader_2.54mm:PinHeader_1x01_P2.54mm_Vertical -> Connector_PinHeader_2.54mm:PinHeader_1x03_P2.54mm_Vertical
Changed lines of the file:
@@
 F 0 "TP2" H 7016 5975 50  0000 C CNN
 F 1 "Test_i2C" H 7016 5884 50  0000 C CNN
-F 2 "Connector_PinHeader_2.54mm:PinHeader_1x01_P2.54mm_Vertical" H 7150 5850 50  0001 C CNN
+F 2 "Connector_PinHeader_2.54mm:PinHeader_1x03_P2.54mm_Vertical" H 7150 5850 50  0001 C CNN
 F 3 "~" H 7150 5850 50  0001 C CNN
 	1    7100 5650

Commit message: first pcb v1.0
Parts:
- added C8, C9: 10uF, Capacitor_SMD:C_0805_2012Metric_Pad1.15x1.40mm_HandSolder, symbol Device:C
- added J15, J16, J17, J18: hole, MountingHole:MountingHole_3.2mm_M3, symbol Connector:Conn_01x01_Female
- added TP7: Test_UART, Connector_PinHeader_2.54mm:PinHeader_1x03_P2.54mm_Vertical, symbol Test_points:Test_UART
Connections:
- net labels added: GNDPWR
- wire segments 111 -> 115
- no-connect marks 0 -> 17
