File: kicad/esp8266.sch (KiCad schematic (older format))
At the start: 42 parts, among them J10 Green, J11 Blue, J12 White, J13 IO_RGBW, J14 +12V, J15 hole, J16 hole, J17 hole, J18 hole, J2 5 / 12V, J3 CONN FT232RL, J4 RJ12-I2C, J5 RJ12-I2C, J6 Onewire, J7 Onewire, J8 Red, J9 Pad, Q1 BSP75, Q2 BSP75, Q3 BSP75, Q4 BSP75, SW1 RESET, SW2 PROG, U1 ESP-12E, U4 MS5637, U6 Si7020-A20, U7 DS18B20

Commit message: add distances
Other:
- note added: "18.01.2019"
- note added: "ESP-12e playground"
Changed lines of the file:
@@
 NoConn ~ 1000 3050
 NoConn ~ 1000 3200
+Text Notes 7400 7500 0    50   ~ 0
+ESP-12e playground
+Text Notes 8150 7650 0    50   ~ 0
+18.01.2019
 $EndSCHEMATC

Commit message: move 3d models to shared library
Parts:
- U4: footprint libs:MS5637 -> hackuarium:MS5637
Changed lines of the file:
@@
 F 0 "U4" H 8450 5937 60  0000 C CNN
 F 1 "MS5637" H 8450 5831 60  0000 C CNN
-F 2 "libs:MS5637" H 8150 5550 60  0001 C CNN
+F 2 "hackuarium:MS5637" H 8150 5550 60  0001 C CNN
 F 3 "" H 8150 5550 60  0000 C CNN
 	1    8450 5600

Commit message: move sub schemas
Changed lines of the file:
@@
 U 5C3A17E5
 F0 "MCP73831" 50
-F1 "MCP73831.sch" 50
+F1 "schemas/MCP73831.sch" 50
 F2 "VIN" I L 3300 1950 50
 F3 "VOUT" O R 4700 1650 50
@@
 U 5C3A2732
 F0 "MCP1703-33" 50
-F1 "mcp1703-33.sch" 50
+F1 "schemas/MCP1703-33.sch" 50
 F2 "VDD" I L 5850 1650 50
 F3 "3.3V" O R 6800 1650 50
@@
 U 5C3D1997
 F0 "MCP1703-50" 50
-F1 "mcp1703-50.sch" 50
+F1 "schemas/MCP1703-50.sch" 50
 F2 "VDD" I L 850 1650 50
 F3 "5.0V" O R 1800 1650 50
