File: kicad/esp8266.sch (KiCad schematic (older format))
At the start: 42 parts, among them J10 Green, J11 Blue, J12 White, J13 IO_RGBW, J14 +12V, J15 hole, J16 hole, J17 hole, J18 hole, J2 5 / 12V, J3 CONN FT232RL, J4 RJ12-I2C, J5 RJ12-I2C, J6 Onewire, J7 Onewire, J8 Red, J9 Pad, Q1 BSP75, Q2 BSP75, Q3 BSP75, Q4 BSP75, SW1 RESET, SW2 PROG, U1 ESP-12E, U4 MS5637, U6 Si7020-A20, U7 DS18B20

Commit message: fix resistor on IO15 and button
Parts:
- added R11: 10k, Resistor_SMD:R_0805_2012Metric_Pad1.15x1.40mm_HandSolder, symbol Device:R
- SW1, SW2: footprint digikey-footprints:Switch_Tactile_SMD_6x6mm -> Button_Switch_SMD:SW_SPST_PTS645
Connections:
- wire segments 115 -> 116
Changed lines of the file:
@@
 F 0 "SW1" H 3500 4535 50  0000 C CNN
 F 1 "RESET" H 3500 4444 50  0000 C CNN
-F 2 "digikey-footprints:Switch_Tactile_SMD_6x6mm" H 3500 4450 50  0001 C CNN
+F 2 "Button_Switch_SMD:SW_SPST_PTS645" H 3500 4450 50  0001 C CNN
 F 3 "" H 3500 4450 50  0001 C CNN
 	1    3500 4250
@@
 F 0 "SW2" H 6200 4535 50  0000 C CNN
 F 1 "PROG" H 6200 4444 50  0000 C CNN
-F 2 "digikey-footprints:Switch_Tactile_SMD_6x6mm" H 6200 4450 50  0001 C CNN
+F 2 "Button_Switch_SMD:SW_SPST_PTS645" H 6200 4450 50  0001 C CNN
 F 3 "" H 6200 4450 50  0001 C CNN
 	1    6200 4250
@@
 Wire Wire Line
 	5250 5050 5600 5050
-Wire Wire Line
-	5250 5150 5600 5150
 Text Notes 5650 4450 0    50   ~ 0
 Onewire\n
@@
 Text Notes 8150 7650 0    50   ~ 0
 18.01.2019
+$Comp
+L Device:R R11
+U 1 1 5CAD1C9A
+P 5950 5300
+F 0 "R11" H 6020 5346 50  0000 L CNN
+F 1 "10k" H 6020 5255 50  0000 L CNN
+F 2 "Resistor_SMD:R_0805_2012Metric_Pad1.15x1.40mm_HandSolder" V 5880 5300 50  0001 C CNN
+F 3 "~" H 5950 5300 50  0001 C CNN
+	1    5950 5300
+	1    0    0    -1
+$EndComp
+$Comp
+L power:GND #PWR0167
+U 1 1 5CAD1D34
+P 5950 5500
+F 0 "#PWR0167" H 5950 5250 50  0001 C CNN
+F 1 "GND" H 5955 5327 50  0000 C CNN
+F 2 "" H 5950 5500 50  0001 C CNN
+F 3 "" H 5950 5500 50  0001 C CNN
+	1    5950 5500
+	1    0    0    -1
+$EndComp
+Wire Wire Line
+	5250 5150 5950 5150
+Wire Wire Line
+	5950 5450 5950 5500
 $EndSCHEMATC
